File: AvrTimer.kicad_sch (KiCad schematic)
At the start: 40 parts, among them Q1 BC846, Q10 BC557, Q11 BC557, Q12 BC557, Q2 BC846, Q3 BC846, Q4 BC846, Q5 BC846, Q6 BC846, Q7 BC846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

Commit message: Partly update scheme for hand-soldering
Parts:
- D4, D5, D6: footprint Diode_SMD:D_1210_3225Metric -> Diode_SMD:D_1210_3225Metric_Pad1.42x2.65mm_HandSolder
- Led1, Led2, Led3: footprint LED_SMD:LED_1210_3225Metric -> LED_SMD:LED_1210_3225Metric_Pad1.42x2.65mm_HandSolder
- Led4: footprint Diode_SMD:D_1210_3225Metric -> LED_SMD:LED_1210_3225Metric_Pad1.42x2.65mm_HandSolder
- Q1, Q10, Q11, Q12, Q2, Q3, Q4, Q5, Q6, Q7, Q8, Q9: footprint Package_TO_SOT_SMD:SOT-23 -> Package_TO_SOT_SMD:SOT-23_Handsoldering

Commit message: Update all footprints to correct ones
Parts:
- Mechanic1: footprint Connector_PinSocket_2.54mm:PinSocket_1x06_P2.54mm_Vertical -> Connector_JST:JST_XH_B6B-XH-A_1x06_P2.50mm_Vertical
- R1, R10, R11, R12, R13, R14, R15, R16, R2, R3, R4, R5, R6, R7, R8, R9: footprint Resistor_SMD:R_1206_3216Metric -> Resistor_SMD:R_1206_3216Metric_Pad1.30x1.75mm_HandSolder
- Serial1: footprint Connector_PinSocket_2.54mm:PinSocket_1x06_P2.54mm_Vertical -> Connector_PinHeader_2.54mm:PinHeader_1x06_P2.54mm_Vertical

Commit message: Update after Alexander's Y. review
Connections:
- net GND: now also Led2.1 (K); no longer R15.2
- net at Controller1.23 (PC0): now also Q11.2 (B); no longer Q12.2 (B)
- net at Controller1.25 (PC2): now also Q12.2 (B); no longer Q11.2 (B)
- net at Mechanic1.6 (Pin_6), Q1.2 (E), R14.1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: now also R15.1; no longer Led2.2 (A)
- new net: Led2.2 (A), R15.2
Other:
- moved on the sheet: Led2, R15
Changed lines of the file:
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@@
     (stroke (width 0) (type solid) (color 0 0 0 0))
   )
-  (wire (pts (xy 165.1 151.13) (xy 261.62 151.13))
+  (wire (pts (xy 165.1 151.13) (xy 252.73 151.13))
     (stroke (width 0) (type solid) (color 0 0 0 0))
   )
@@
     (stroke (width 0) (type solid) (color 0 0 0 0))
   )
+  (wire (pts (xy 252.73 132.08) (xy 252.73 151.13))
+    (stroke (width 0) (type solid) (color 0 0 0 0))
+  )
+  (wire (pts (xy 252.73 132.08) (xy 261.62 132.08))
+    (stroke (width 0) (type solid) (color 0 0 0 0))
+  )
   (wire (pts (xy 255.27 115.57) (xy 261.62 115.57))
     (stroke (width 0) (type solid) (color 0 0 0 0))
@@
     (stroke (width 0) (type solid) (color 0 0 0 0))
   )
-  (wire (pts (xy 256.54 132.08) (xy 261.62 132.08))
-    (stroke (width 0) (type solid) (color 0 0 0 0))
-  )
-  (wire (pts (xy 256.54 153.67) (xy 256.54 132.08))
+  (wire (pts (xy 256.54 151.13) (xy 261.62 151.13))
+    (stroke (width 0) (type solid) (color 0 0 0 0))
+  )
+  (wire (pts (xy 256.54 153.67) (xy 256.54 151.13))
     (stroke (width 0) (type solid) (color 0 0 0 0))
   )
@@
     (pin "2")
   )
-  (symbol (lib_id "AvrTimer-rescue:R-Device") (at 74.93 100.33 0) (mirror y) (unit 1)
-    (in_bom yes) (on_board yes)
-    (property "Reference" "R15" (id 0) (at 73.152 99.1616 0)
-      (effects (font (size 1.27 1.27)) (justify left))
-    )
-    (property "Value" "R" (id 1) (at 73.152 101.473 0)
-      (effects (font (size 1.27 1.27)) (justify left))
-    )
-    (property "Footprint" "Resistor_SMD:R_1206_3216Metric_Pad1.30x1.75mm_HandSolder" (id 2) (at 76.708 100.33 90)
-      (effects (font (size 1.27 1.27)) hide)
-    )
-    (property "Datasheet" "~" (id 3) (at 74.93 100.33 0)
+  (symbol (lib_id "AvrTimer-rescue:R-Device") (at 74.93 92.71 0) (unit 1)
+    (in_bom yes) (on_board yes)
+    (property "Reference" "R15" (id 0) (at 76.708 91.5416 0)
+      (effects (font (size 1.27 1.27)) (justify left))
+    )
+    (property "Value" "R" (id 1) (at 76.708 93.853 0)
+      (effects (font (size 1.27 1.27)) (justify left))
+    )
+    (property "Footprint" "Resistor_SMD:R_1206_3216Metric_Pad1.30x1.75mm_HandSolder" (id 2) (at 73.152 92.71 90)
+      (effects (font (size 1.27 1.27)) hide)
+    )
+    (property "Datasheet" "~" (id 3) (at 74.93 92.71 0)
       (effects (font (size 1.27 1.27)) hide)
     )
@@
     (pin "2")
   )
-  (symbol (lib_id "AvrTimer-rescue:LED-Device") (at 74.93 92.71 270) (mirror x) (unit 1)
-    (in_bom yes) (on_board yes)
-    (property "Reference" "Led2" (id 0) (at 80.4418 92.8878 0))
-    (property "Value" "Red" (id 1) (at 78.1304 92.8878 0))
-    (property "Footprint" "LED_SMD:LED_1210_3225Metric_Pad1.42x2.65mm_HandSolder" (id 2) (at 74.93 92.71 0)
-      (effects (font (size 1.27 1.27)) hide)
-    )
-    (property "Datasheet" "~" (id 3) (at 74.93 92.71 0)
-      (effects (font (size 1.27 1.27)) hide)
-    )
+  (symbol (lib_id "AvrTimer-rescue:LED-Device") (at 74.93 100.33 90) (unit 1)
+    (in_bom yes) (on_board yes)
+    (property "Reference" "Led2" (id 0) (at 69.4182 100.5078 0))
+    (property "Value" "Red" (id 1) (at 71.7296 100.5078 0))
+    (property "Footprint" "LED_SMD:LED_1210_3225Metric_Pad1.42x2.65mm_HandSolder" (id 2) (at 74.93 100.33 0)
+      (effects (font (size 1.27 1.27)) hide)
+    )
+    (property "Datasheet" "~" (id 3) (at 74.93 100.33 0)
+      (effects (font (size 1.27 1.27)) hide)
+    )

Commit message: Final version of base board
Connections:
- net GND: now also Controller1.22 (AGND)
- net VCC: now also Controller1.20 (AVCC)
- no-connect marks 6 -> 8
Changed lines of the file:
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@@
   (junction (at 90.17 139.7) (diameter 1.016) (color 0 0 0 0))
   (junction (at 97.79 63.5) (diameter 1.016) (color 0 0 0 0))
+  (junction (at 133.35 50.8) (diameter 1.016) (color 0 0 0 0))
   (junction (at 157.48 71.12) (diameter 1.016) (color 0 0 0 0))
   (junction (at 158.75 73.66) (diameter 1.016) (color 0 0 0 0))
@@
   (junction (at 173.99 100.33) (diameter 1.016) (color 0 0 0 0))
   (junction (at 173.99 114.3) (diameter 1.016) (color 0 0 0 0))
+  (no_connect (at 118.11 78.74))
   (no_connect (at 148.59 99.06))
   (no_connect (at 148.59 101.6))
@@
   (no_connect (at 148.59 111.76))
   (no_connect (at 148.59 114.3))
+  (no_connect (at 148.59 116.84))
   (no_connect (at 228.6 86.36))
   (wire (pts (xy 22.86 46.99) (xy 22.86 52.07))
@@
     (stroke (width 0) (type solid) (color 0 0 0 0))
   )
+  (wire (pts (xy 45.72 34.29) (xy 50.8 34.29))
+    (stroke (width 0) (type solid) (color 0 0 0 0))
+  )
   (wire (pts (xy 45.72 38.1) (xy 45.72 64.77))
     (stroke (width 0) (type solid) (color 0 0 0 0))
@@
     (stroke (width 0) (type solid) (color 0 0 0 0))
   )
-  (wire (pts (xy 49.53 34.29) (xy 45.72 34.29))
-    (stroke (width 0) (type solid) (color 0 0 0 0))
-  )
-  (wire (pts (xy 49.53 38.1) (xy 49.53 34.29))
-    (stroke (width 0) (type solid) (color 0 0 0 0))
-  )
   (wire (pts (xy 50.8 31.75) (xy 50.8 33.02))
     (stroke (width 0) (type solid) (color 0 0 0 0))
   )
-  (wire (pts (xy 50.8 38.1) (xy 49.53 38.1))
-    (stroke (width 0) (type solid) (color 0 0 0 0))
-  )
-  (wire (pts (xy 50.8 38.1) (xy 50.8 69.85))
+  (wire (pts (xy 50.8 34.29) (xy 50.8 69.85))
     (stroke (width 0) (type solid) (color 0 0 0 0))
   )
@@
     (stroke (width 0) (type solid) (color 0 0 0 0))
   )
-  (wire (pts (xy 133.35 55.88) (xy 133.35 22.86))
+  (wire (pts (xy 133.35 50.8) (xy 133.35 22.86))
+    (stroke (width 0) (type solid) (color 0 0 0 0))
+  )
+  (wire (pts (xy 133.35 50.8) (xy 135.89 50.8))
+    (stroke (width 0) (type solid) (color 0 0 0 0))
+  )
+  (wire (pts (xy 133.35 55.88) (xy 133.35 50.8))
+    (stroke (width 0) (type solid) (color 0 0 0 0))
+  )
+  (wire (pts (xy 135.89 50.8) (xy 135.89 55.88))
     (stroke (width 0) (type solid) (color 0 0 0 0))
   )
@@
     )
     (property "Datasheet" "" (id 3) (at 133.35 127 0)
+      (effects (font (size 1.27 1.27)) hide)
+    )
+    (pin "1")
+  )
+  (symbol (lib_id "power:GND") (at 135.89 127 0) (unit 1)
+    (in_bom yes) (on_board yes) (fields_autoplaced)
+    (property "Reference" "#PWR?" (id 0) (at 135.89 133.35 0)
+      (effects (font (size 1.27 1.27)) hide)
+    )
+    (property "Value" "GND" (id 1) (at 135.89 132.08 0))
+    (property "Footprint" "" (id 2) (at 135.89 127 0)
+      (effects (font (size 1.27 1.27)) hide)
+    )
+    (property "Datasheet" "" (id 3) (at 135.89 127 0)
       (effects (font (size 1.27 1.27)) hide)
     )
@@
       (reference "#PWR0109") (unit 1) (value "GND") (footprint "")
     )
+    (path "/d917b3d2-6947-425b-a61f-7f88b12a6326"
+      (reference "#PWR?") (unit 1) (value "GND") (footprint "")
+    )
     (path "/00000000-0000-0000-0000-00006245e17b"
