File: pcb/base/AvrTimer-Base.kicad_pcb (KiCad board)
At the start: 2 copper layers, 67 x 48.5 mm, 43 parts, among them Q1 BC846, Q10 BC557, Q11 BC557, Q12 BC557, Q2 BC846, Q3 BC846, Q4 BC846, Q5 BC846, Q6 BC846, Q7 BC846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

Commit message: Add local pretty library
Add source reference and board name o Base board
Parts:
- Display1: footprint AvrTimer:BC56-12GWA -> Footprints:BC56-12GWA
Other:
- board text added: "Base Board"
- board text added: "github.com/ein-shved/AvrTimer"

Commit message: Replace diode footprints to shop real ones
Parts:
- D4, D5, D6: footprint Diode_SMD:D_1210_3225Metric_Pad1.42x2.65mm_HandSolder -> Diode_SMD:D_SOD-123F
