File: pcb/base/AvrTimer-Base.kicad_sch (KiCad schematic)
At the start: 40 parts, among them Q1 BC846, Q10 BC557, Q11 BC557, Q12 BC557, Q2 BC846, Q3 BC846, Q4 BC846, Q5 BC846, Q6 BC846, Q7 BC846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

Commit message: Add local pretty library
Add source reference and board name o Base board
Parts:
- Display1: footprint AvrTimer:BC56-12GWA -> Footprints:BC56-12GWA
Changed lines of the file:
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@@
   (symbol (lib_id "power:GND") (at 135.89 127 0) (unit 1)
     (in_bom yes) (on_board yes) (fields_autoplaced)
-    (property "Reference" "#PWR?" (id 0) (at 135.89 133.35 0)
+    (property "Reference" "#PWR0110" (id 0) (at 135.89 133.35 0)
       (effects (font (size 1.27 1.27)) hide)
     )
@@
       (effects (font (size 1.524 1.524)))
     )
-    (property "Footprint" "AvrTimer:BC56-12GWA" (id 2) (at 248.92 67.564 0)
+    (property "Footprint" "Footprints:BC56-12GWA" (id 2) (at 248.92 67.564 0)
       (effects (font (size 1.524 1.524)) hide)
     )
@@
     )
     (path "/d917b3d2-6947-425b-a61f-7f88b12a6326"
-      (reference "#PWR?") (unit 1) (value "GND") (footprint "")
+      (reference "#PWR0110") (unit 1) (value "GND") (footprint "")
     )
     (path "/00000000-0000-0000-0000-00006245e17b"
@@
     )
     (path "/00000000-0000-0000-0000-00006249ae87"
-      (reference "Display1") (unit 1) (value "BC56-12SRWA") (footprint "AvrTimer:BC56-12GWA")
+      (reference "Display1") (unit 1) (value "BC56-12SRWA") (footprint "Footprints:BC56-12GWA")
     )
     (path "/00000000-0000-0000-0000-000062989eec"

Commit message: Replace diode footprints to shop real ones
Parts:
- D4, D5, D6: footprint Diode_SMD:D_1210_3225Metric_Pad1.42x2.65mm_HandSolder -> Diode_SMD:D_SOD-123F
Changed lines of the file:
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@@
     (property "Reference" "D4" (id 0) (at 80.01 115.1382 0))
     (property "Value" "D" (id 1) (at 80.01 117.4496 0))
-    (property "Footprint" "Diode_SMD:D_1210_3225Metric_Pad1.42x2.65mm_HandSolder" (id 2) (at 80.01 120.65 0)
+    (property "Footprint" "Diode_SMD:D_SOD-123F" (id 2) (at 80.01 120.65 0)
       (effects (font (size 1.27 1.27)) hide)
     )
@@
     (property "Reference" "D5" (id 0) (at 80.01 125.2982 0))
     (property "Value" "D" (id 1) (at 80.01 127.6096 0))
-    (property "Footprint" "Diode_SMD:D_1210_3225Metric_Pad1.42x2.65mm_HandSolder" (id 2) (at 80.01 130.81 0)
+    (property "Footprint" "Diode_SMD:D_SOD-123F" (id 2) (at 80.01 130.81 0)
       (effects (font (size 1.27 1.27)) hide)
     )
@@
     (property "Reference" "D6" (id 0) (at 80.01 134.1882 0))
     (property "Value" "D" (id 1) (at 80.01 136.4996 0))
-    (property "Footprint" "Diode_SMD:D_1210_3225Metric_Pad1.42x2.65mm_HandSolder" (id 2) (at 80.01 139.7 0)
+    (property "Footprint" "Diode_SMD:D_SOD-123F" (id 2) (at 80.01 139.7 0)
       (effects (font (size 1.27 1.27)) hide)
     )
@@
     )
     (path "/00000000-0000-0000-0000-000062739cdf"
-      (reference "D4") (unit 1) (value "D") (footprint "Diode_SMD:D_1210_3225Metric_Pad1.42x2.65mm_HandSolder")
+      (reference "D4") (unit 1) (value "D") (footprint "Diode_SMD:D_SOD-123F")
     )
     (path "/00000000-0000-0000-0000-00006272fe3e"
-      (reference "D5") (unit 1) (value "D") (footprint "Diode_SMD:D_1210_3225Metric_Pad1.42x2.65mm_HandSolder")
+      (reference "D5") (unit 1) (value "D") (footprint "Diode_SMD:D_SOD-123F")
     )
     (path "/00000000-0000-0000-0000-00006272d335"
-      (reference "D6") (unit 1) (value "D") (footprint "Diode_SMD:D_1210_3225Metric_Pad1.42x2.65mm_HandSolder")
+      (reference "D6") (unit 1) (value "D") (footprint "Diode_SMD:D_SOD-123F")
     )
     (path "/00000000-0000-0000-0000-00006249ae87"

Commit message: [PCB] Add values for R and C
Parts:
- R1, R2, R3, R4: value R -> 10 kOhm
- R10, R11, R12, R13, R6, R7, R8, R9: value R -> 300 Ohm
- R14, R15, R16, R5: value R -> 150 Ohm
