File: pcb/mech/AvrTimer-Mech.kicad_sch (KiCad schematic)
At the start: 24 parts, among them J1 USB_B_Micro, Q1 BC846, SW1 SW_DIP_x01, SW2 SW_DIP_x01, SW3 SW_DIP_x01, SW4 SW_DPDT_x2, SW5 SW_DIP_x02, U1 L7805

Commit message: Replace diode footprints to shop real ones
Parts:
- D1, D2, D3: footprint Diode_SMD:D_1210_3225Metric_Pad1.42x2.65mm_HandSolder -> Diode_SMD:D_SOD-123F
Changed lines of the file:
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@@
     (property "Reference" "D1" (id 0) (at 76.2 27.305 0))
     (property "Value" "DIODE" (id 1) (at 76.2 29.845 0))
-    (property "Footprint" "Diode_SMD:D_1210_3225Metric_Pad1.42x2.65mm_HandSolder" (id 2) (at 76.2 34.925 0)
+    (property "Footprint" "Diode_SMD:D_SOD-123F" (id 2) (at 76.2 34.925 0)
       (effects (font (size 1.27 1.27)) hide)
     )
@@
     (property "Reference" "D2" (id 0) (at 106.68 19.685 0))
     (property "Value" "DIODE" (id 1) (at 116.84 20.955 0))
-    (property "Footprint" "Diode_SMD:D_1210_3225Metric_Pad1.42x2.65mm_HandSolder" (id 2) (at 109.22 23.495 0)
+    (property "Footprint" "Diode_SMD:D_SOD-123F" (id 2) (at 109.22 23.495 0)
       (effects (font (size 1.27 1.27)) hide)
     )
@@
     (property "Reference" "D3" (id 0) (at 170.18 52.07 0))
     (property "Value" "DIODE" (id 1) (at 171.45 55.88 0))
-    (property "Footprint" "Diode_SMD:D_1210_3225Metric_Pad1.42x2.65mm_HandSolder" (id 2) (at 171.45 60.96 0)
+    (property "Footprint" "Diode_SMD:D_SOD-123F" (id 2) (at 171.45 60.96 0)
       (effects (font (size 1.27 1.27)) hide)
     )
@@
     )
     (path "/f3ef0f38-6c02-44eb-89f4-36c971010a05"
-      (reference "D1") (unit 1) (value "DIODE") (footprint "Diode_SMD:D_1210_3225Metric_Pad1.42x2.65mm_HandSolder")
+      (reference "D1") (unit 1) (value "DIODE") (footprint "Diode_SMD:D_SOD-123F")
     )
     (path "/e9eb0cf1-7cfc-481d-aede-5ccf2b2563b5"
-      (reference "D2") (unit 1) (value "DIODE") (footprint "Diode_SMD:D_1210_3225Metric_Pad1.42x2.65mm_HandSolder")
+      (reference "D2") (unit 1) (value "DIODE") (footprint "Diode_SMD:D_SOD-123F")
     )
     (path "/98e49acb-d0fe-43d8-8f2f-43c384e363c5"
-      (reference "D3") (unit 1) (value "DIODE") (footprint "Diode_SMD:D_1210_3225Metric_Pad1.42x2.65mm_HandSolder")
+      (reference "D3") (unit 1) (value "DIODE") (footprint "Diode_SMD:D_SOD-123F")
     )
     (path "/5e68ff61-6a09-45cc-8df6-d7521682d52c"

Commit message: Update after Alexander's review
Change-Id: Ia4ad441f5e963f780b6a0a3a3c0dc55fa8eb64d7
Parts:
- added C5, C6: C, Capacitor_SMD:C_0402_1005Metric_Pad0.74x0.62mm_HandSolder, symbol Device:C
- added R6: R, Resistor_SMD:R_1206_3216Metric_Pad1.30x1.75mm_HandSolder, symbol Device:R
Connections:
- net GND: now also C5.1, C6.1, R6.1
- net at J1.6 (Shield): now also C5.2, C6.2, R6.2
- no-connect marks 5 -> 4
Changed lines of the file:
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@@
   (junction (at 132.08 34.925) (diameter 0.9144) (color 0 0 0 0))
   (junction (at 152.4 60.96) (diameter 0.9144) (color 0 0 0 0))
+  (junction (at 198.12 33.02) (diameter 0.9144) (color 0 0 0 0))
+  (junction (at 198.12 46.99) (diameter 0.9144) (color 0 0 0 0))
   (no_connect (at 67.945 34.925))
   (no_connect (at 187.96 63.5))
   (no_connect (at 187.96 66.04))
   (no_connect (at 187.96 68.58))
-  (no_connect (at 198.12 58.42))
   (wire (pts (xy 54.61 40.005) (xy 54.61 46.355))
     (stroke (width 0) (type solid) (color 0 0 0 0))
@@
     (stroke (width 0) (type solid) (color 0 0 0 0))
   )
+  (wire (pts (xy 187.96 33.02) (xy 198.12 33.02))
+    (stroke (width 0) (type solid) (color 0 0 0 0))
+  )
+  (wire (pts (xy 187.96 36.83) (xy 187.96 33.02))
+    (stroke (width 0) (type solid) (color 0 0 0 0))
+  )
+  (wire (pts (xy 187.96 44.45) (xy 187.96 46.99))
+    (stroke (width 0) (type solid) (color 0 0 0 0))
+  )
+  (wire (pts (xy 187.96 46.99) (xy 198.12 46.99))
+    (stroke (width 0) (type solid) (color 0 0 0 0))
+  )
   (wire (pts (xy 187.96 73.66) (xy 181.61 73.66))
+    (stroke (width 0) (type solid) (color 0 0 0 0))
+  )
+  (wire (pts (xy 198.12 33.02) (xy 198.12 36.83))
+    (stroke (width 0) (type solid) (color 0 0 0 0))
+  )
+  (wire (pts (xy 198.12 33.02) (xy 209.55 33.02))
+    (stroke (width 0) (type solid) (color 0 0 0 0))
+  )
+  (wire (pts (xy 198.12 44.45) (xy 198.12 46.99))
+    (stroke (width 0) (type solid) (color 0 0 0 0))
+  )
+  (wire (pts (xy 198.12 46.99) (xy 198.12 58.42))
+    (stroke (width 0) (type solid) (color 0 0 0 0))
+  )
+  (wire (pts (xy 198.12 46.99) (xy 209.55 46.99))
+    (stroke (width 0) (type solid) (color 0 0 0 0))
+  )
+  (wire (pts (xy 209.55 33.02) (xy 209.55 36.83))
+    (stroke (width 0) (type solid) (color 0 0 0 0))
+  )
+  (wire (pts (xy 209.55 46.99) (xy 209.55 44.45))
     (stroke (width 0) (type solid) (color 0 0 0 0))
   )
@@
     )
     (property "Datasheet" "" (id 3) (at 195.58 58.42 0)
+      (effects (font (size 1.27 1.27)) hide)
+    )
+    (pin "1")
+  )
+  (symbol (lib_id "power:GND") (at 198.12 33.02 180) (unit 1)
+    (in_bom yes) (on_board yes) (fields_autoplaced)
+    (property "Reference" "#PWR010" (id 0) (at 198.12 26.67 0)
+      (effects (font (size 1.27 1.27)) hide)
+    )
+    (property "Value" "GND" (id 1) (at 198.12 27.94 0))
+    (property "Footprint" "" (id 2) (at 198.12 33.02 0)
+      (effects (font (size 1.27 1.27)) hide)
+    )
+    (property "Datasheet" "" (id 3) (at 198.12 33.02 0)
       (effects (font (size 1.27 1.27)) hide)
     )
@@
     (pin "2")
   )
+  (symbol (lib_id "Device:R") (at 187.96 40.64 0) (unit 1)
+    (in_bom yes) (on_board yes) (fields_autoplaced)
+    (property "Reference" "R6" (id 0) (at 190.5 39.3699 0)
+      (effects (font (size 1.27 1.27)) (justify left))
+    )
+    (property "Value" "R" (id 1) (at 190.5 41.9099 0)
+      (effects (font (size 1.27 1.27)) (justify left))
+    )
+    (property "Footprint" "Resistor_SMD:R_1206_3216Metric_Pad1.30x1.75mm_HandSolder" (id 2) (at 186.182 40.64 90)
+      (effects (font (size 1.27 1.27)) hide)
+    )
+    (property "Datasheet" "~" (id 3) (at 187.96 40.64 0)
+      (effects (font (size 1.27 1.27)) hide)
+    )
+    (pin "1")
+    (pin "2")
+  )
   (symbol (lib_name "Connector_Generic:Conn_01x02_1") (lib_id "Connector_Generic:Conn_01x02") (at 49.53 37.465 0) (mirror y) (unit 1)
     (in_bom yes) (on_board yes)
@@
     )
     (property "Datasheet" "~" (id 3) (at 132.08 42.545 0)
+      (effects (font (size 1.27 1.27)) hide)
+    )
+    (pin "1")
+    (pin "2")
+  )
+  (symbol (lib_id "Device:C") (at 198.12 40.64 0) (unit 1)
+    (in_bom yes) (on_board yes) (fields_autoplaced)
+    (property "Reference" "C5" (id 0) (at 201.93 39.3699 0)
+      (effects (font (size 1.27 1.27)) (justify left))
+    )
+    (property "Value" "C" (id 1) (at 201.93 41.9099 0)
+      (effects (font (size 1.27 1.27)) (justify left))
+    )
+    (property "Footprint" "Capacitor_SMD:C_0402_1005Metric_Pad0.74x0.62mm_HandSolder" (id 2) (at 199.0852 44.45 0)
+      (effects (font (size 1.27 1.27)) hide)
+    )
+    (property "Datasheet" "~" (id 3) (at 198.12 40.64 0)
+      (effects (font (size 1.27 1.27)) hide)
+    )
+    (pin "1")
+    (pin "2")
+  )
+  (symbol (lib_id "Device:C") (at 209.55 40.64 0) (unit 1)
+    (in_bom yes) (on_board yes) (fields_autoplaced)
+    (property "Reference" "C6" (id 0) (at 213.36 39.3699 0)
+      (effects (font (size 1.27 1.27)) (justify left))
+    )
+    (property "Value" "C" (id 1) (at 213.36 41.9099 0)
+      (effects (font (size 1.27 1.27)) (justify left))
+    )
+    (property "Footprint" "Capacitor_SMD:C_0402_1005Metric_Pad0.74x0.62mm_HandSolder" (id 2) (at 210.5152 44.45 0)
+      (effects (font (size 1.27 1.27)) hide)
+    )
+    (property "Datasheet" "~" (id 3) (at 209.55 40.64 0)
       (effects (font (size 1.27 1.27)) hide)
     )
@@
       (reference "#PWR09") (unit 1) (value "GND") (footprint "")
     )
+    (path "/42d56a7d-17d9-4d0a-af31-1ad4ef2ccada"
+      (reference "#PWR010") (unit 1) (value "GND") (footprint "")
+    )
     (path "/e6ddafb7-2fdf-49be-b3d6-d13ed97c6af4"
       (reference "BZ1") (unit 1) (value "Buzzer") (footprint "Buzzer_Beeper:Buzzer_12x9.5RM7.6")
@@
       (reference "C4") (unit 1) (value "C_Polarized") (footprint "Capacitor_THT:CP_Radial_D10.0mm_P5.00mm")
     )
+    (path "/6cda93ea-becc-43f0-b134-cdec720d5bdd"
+      (reference "C5") (unit 1) (value "C") (footprint "Capacitor_SMD:C_0402_1005Metric_Pad0.74x0.62mm_HandSolder")
+    )
+    (path "/db7a4956-fc0d-4800-95e8-913d6f049d8b"
+      (reference "C6") (unit 1) (value "C") (footprint "Capacitor_SMD:C_0402_1005Metric_Pad0.74x0.62mm_HandSolder")
+    )
     (path "/f3ef0f38-6c02-44eb-89f4-36c971010a05"
       (reference "D1") (unit 1) (value "DIODE") (footprint "Diode_SMD:D_SOD-123F")
@@
       (reference "R5") (unit 1) (value "R") (footprint "Resistor_SMD:R_1206_3216Metric_Pad1.30x1.75mm_HandSolder")
     )
+    (path "/b11245bd-4cec-48a7-9ad9-f656499448a0"
+      (reference "R6") (unit 1) (value "R") (footprint "Resistor_SMD:R_1206_3216Metric_Pad1.30x1.75mm_HandSolder")
+    )
     (path "/87ead37c-f275-4b39-8c0d-c36556ce8fdc"

Commit message: [PCB] Add values for R and C
Parts:
- C1: value C_Polarized -> 470 uF
- C2, C3, C5: value C -> 100 nF
- C4: value C_Polarized -> 10 uF
- C6: value C -> 1 nF
- R1, R2, R3: value R -> 10 kOhm
- R4: value R -> 100 Ohm
- R5: value R -> 10 Ohm
- R6: value R -> 1 MOhm
Changed lines of the file:
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@@
   )
   (symbol (lib_id "Device:R") (at 77.47 102.87 90) (unit 1)
-    (in_bom yes) (on_board yes) (fields_autoplaced)
+    (in_bom yes) (on_board yes)
     (property "Reference" "R1" (id 0) (at 77.47 96.52 90))
-    (property "Value" "R" (id 1) (at 77.47 99.06 90))
+    (property "Value" "10 kOhm" (id 1) (at 78.74 99.06 90))
     (property "Footprint" "Resistor_SMD:R_1206_3216Metric_Pad1.30x1.75mm_HandSolder" (id 2) (at 77.47 104.648 90)
       (effects (font (size 1.27 1.27)) hide)
@@
   )
   (symbol (lib_id "Device:R") (at 92.71 102.87 90) (unit 1)
-    (in_bom yes) (on_board yes) (fields_autoplaced)
+    (in_bom yes) (on_board yes)
     (property "Reference" "R2" (id 0) (at 92.71 96.52 90))
-    (property "Value" "R" (id 1) (at 92.71 99.06 90))
+    (property "Value" "10 kOhm" (id 1) (at 91.44 99.06 90))
     (property "Footprint" "Resistor_SMD:R_1206_3216Metric_Pad1.30x1.75mm_HandSolder" (id 2) (at 92.71 104.648 90)
       (effects (font (size 1.27 1.27)) hide)
@@
   )
   (symbol (lib_id "Device:R") (at 106.68 102.87 90) (unit 1)
-    (in_bom yes) (on_board yes) (fields_autoplaced)
+    (in_bom yes) (on_board yes)
     (property "Reference" "R3" (id 0) (at 106.68 96.52 90))
-    (property "Value" "R" (id 1) (at 106.68 99.06 90))
+    (property "Value" "10 kOhm" (id 1) (at 105.41 99.06 90))
     (property "Footprint" "Resistor_SMD:R_1206_3216Metric_Pad1.30x1.75mm_HandSolder" (id 2) (at 106.68 104.648 90)
       (effects (font (size 1.27 1.27)) hide)
@@
       (effects (font (size 1.27 1.27)) (justify right))
     )
-    (property "Value" "R" (id 1) (at 142.24 83.8199 0)
+    (property "Value" "10 Ohm" (id 1) (at 142.24 83.8199 0)
       (effects (font (size 1.27 1.27)) (justify right))
     )
@@
     (in_bom yes) (on_board yes)
     (property "Reference" "R4" (id 0) (at 156.21 83.82 90))
-    (property "Value" "R" (id 1) (at 156.21 80.01 90))
+    (property "Value" "100 Ohm" (id 1) (at 161.29 85.09 90))
     (property "Footprint" "Resistor_SMD:R_1206_3216Metric_Pad1.30x1.75mm_HandSolder" (id 2) (at 160.528 81.915 90)
       (effects (font (size 1.27 1.27)) hide)
@@
       (effects (font (size 1.27 1.27)) (justify left))
     )
-    (property "Value" "R" (id 1) (at 190.5 41.9099 0)
+    (property "Value" "1 MOhm" (id 1) (at 190.5 41.9099 0)
       (effects (font (size 1.27 1.27)) (justify left))
     )
@@
       (effects (font (size 1.27 1.27)) (justify left))
     )
-    (property "Value" "C_Polarized" (id 1) (at 74.93 45.0849 0)
+    (property "Value" "470 uF" (id 1) (at 74.93 45.0849 0)
       (effects (font (size 1.27 1.27)) (justify left))
     )
@@
       (effects (font (size 1.27 1.27)) (justify left))
     )
-    (property "Value" "C" (id 1) (at 97.79 43.8149 0)
+    (property "Value" "100 nF" (id 1) (at 97.79 43.8149 0)
       (effects (font (size 1.27 1.27)) (justify left))
     )
@@
       (effects (font (size 1.27 1.27)) (justify left))
     )
-    (property "Value" "C" (id 1) (at 118.11 43.8149 0)
+    (property "Value" "100 nF" (id 1) (at 118.11 43.8149 0)
       (effects (font (size 1.27 1.27)) (justify left))
     )
@@
       (effects (font (size 1.27 1.27)) (justify left))
     )
-    (property "Value" "C_Polarized" (id 1) (at 134.62 45.0849 0)
+    (property "Value" "10 uF" (id 1) (at 134.62 45.0849 0)
       (effects (font (size 1.27 1.27)) (justify left))
     )
@@
       (effects (font (size 1.27 1.27)) (justify left))
     )
-    (property "Value" "C" (id 1) (at 201.93 41.9099 0)
+    (property "Value" "100 nF" (id 1) (at 201.93 41.9099 0)
       (effects (font (size 1.27 1.27)) (justify left))
     )
@@
       (effects (font (size 1.27 1.27)) (justify left))
     )
-    (property "Value" "C" (id 1) (at 213.36 41.9099 0)
+    (property "Value" "1 nF" (id 1) (at 213.36 41.9099 0)
       (effects (font (size 1.27 1.27)) (justify left))
     )
@@
     )
     (path "/294446c2-1f3a-4021-be4d-857ed62a3b7b"
-      (reference "C1") (unit 1) (value "C_Polarized") (footprint "Capacitor_THT:CP_Radial_D10.0mm_P5.00mm")
+      (reference "C1") (unit 1) (value "470 uF") (footprint "Capacitor_THT:CP_Radial_D10.0mm_P5.00mm")
     )
     (path "/646e1802-57ed-4698-8117-e36ed78ae892"
-      (reference "C2") (unit 1) (value "C") (footprint "Capacitor_SMD:C_0402_1005Metric_Pad0.74x0.62mm_HandSolder")
+      (reference "C2") (unit 1) (value "100 nF") (footprint "Capacitor_SMD:C_0402_1005Metric_Pad0.74x0.62mm_HandSolder")
     )
     (path "/c63561dc-6e7b-4bc7-95a6-4f977cd0c8c8"
-      (reference "C3") (unit 1) (value "C") (footprint "Capacitor_SMD:C_0402_1005Metric_Pad0.74x0.62mm_HandSolder")
+      (reference "C3") (unit 1) (value "100 nF") (footprint "Capacitor_SMD:C_0402_1005Metric_Pad0.74x0.62mm_HandSolder")
     )
     (path "/2a527657-ab14-429e-8b1b-53f14d84002f"
-      (reference "C4") (unit 1) (value "C_Polarized") (footprint "Capacitor_THT:CP_Radial_D10.0mm_P5.00mm")
+      (reference "C4") (unit 1) (value "10 uF") (footprint "Capacitor_THT:CP_Radial_D10.0mm_P5.00mm")
     )
     (path "/6cda93ea-becc-43f0-b134-cdec720d5bdd"
-      (reference "C5") (unit 1) (value "C") (footprint "Capacitor_SMD:C_0402_1005Metric_Pad0.74x0.62mm_HandSolder")
+      (reference "C5") (unit 1) (value "100 nF") (footprint "Capacitor_SMD:C_0402_1005Metric_Pad0.74x0.62mm_HandSolder")
     )
     (path "/db7a4956-fc0d-4800-95e8-913d6f049d8b"
-      (reference "C6") (unit 1) (value "C") (footprint "Capacitor_SMD:C_0402_1005Metric_Pad0.74x0.62mm_HandSolder")
+      (reference "C6") (unit 1) (value "1 nF") (footprint "Capacitor_SMD:C_0402_1005Metric_Pad0.74x0.62mm_HandSolder")
     )
     (path "/f3ef0f38-6c02-44eb-89f4-36c971010a05"
@@
     )
     (path "/536c8c1d-8a2c-4c97-98a3-2fa8e32588a1"
-      (reference "R1") (unit 1) (value "R") (footprint "Resistor_SMD:R_1206_3216Metric_Pad1.30x1.75mm_HandSolder")
+      (reference "R1") (unit 1) (value "10 kOhm") (footprint "Resistor_SMD:R_1206_3216Metric_Pad1.30x1.75mm_HandSolder")
     )
     (path "/6806cf43-1e4d-4a12-afde-70af27240296"
-      (reference "R2") (unit 1) (value "R") (footprint "Resistor_SMD:R_1206_3216Metric_Pad1.30x1.75mm_HandSolder")
+      (reference "R2") (unit 1) (value "10 kOhm") (footprint "Resistor_SMD:R_1206_3216Metric_Pad1.30x1.75mm_HandSolder")
     )
     (path "/7e4aa0c2-d54f-4f1e-9148-e8d542f4dd9e"
-      (reference "R3") (unit 1) (value "R") (footprint "Resistor_SMD:R_1206_3216Metric_Pad1.30x1.75mm_HandSolder")
+      (reference "R3") (unit 1) (value "10 kOhm") (footprint "Resistor_SMD:R_1206_3216Metric_Pad1.30x1.75mm_HandSolder")
     )
     (path "/d2e4d1b8-c334-45fd-84ca-cd581b038cd8"
-      (reference "R4") (unit 1) (value "R") (footprint "Resistor_SMD:R_1206_3216Metric_Pad1.30x1.75mm_HandSolder")
+      (reference "R4") (unit 1) (value "100 Ohm") (footprint "Resistor_SMD:R_1206_3216Metric_Pad1.30x1.75mm_HandSolder")
     )
     (path "/889770de-50af-4e11-80bc-31eb7b21fd7d"
-      (reference "R5") (unit 1) (value "R") (footprint "Resistor_SMD:R_1206_3216Metric_Pad1.30x1.75mm_HandSolder")
+      (reference "R5") (unit 1) (value "10 Ohm") (footprint "Resistor_SMD:R_1206_3216Metric_Pad1.30x1.75mm_HandSolder")
     )
     (path "/b11245bd-4cec-48a7-9ad9-f656499448a0"
-      (reference "R6") (unit 1) (value "R") (footprint "Resistor_SMD:R_1206_3216Metric_Pad1.30x1.75mm_HandSolder")
+      (reference "R6") (unit 1) (value "1 MOhm") (footprint "Resistor_SMD:R_1206_3216Metric_Pad1.30x1.75mm_HandSolder")
     )
     (path "/87ead37c-f275-4b39-8c0d-c36556ce8fdc"
